Commit message: add realsense camera to moveit config file

File: ur5_moveit_config/config/gazebo_ur5.urdf (robot description, URDF)
Before this commit: robot ur5, 21 links, 20 joints
Links:
- added link d435_bottom_screw_frame
- added link d435_color_frame
- added link d435_color_optical_frame
- added link d435_depth_frame
- added link d435_depth_optical_frame
- added link d435_left_ir_frame
- added link d435_left_ir_optical_frame
- added link d435_link, mass 0.564; collision box size=0.02505 0.09 0.025; visual mesh filename=package://realsense_ros_gazebo/meshes/realsense_d435.stl
- added link d435_right_ir_frame
- added link d435_right_ir_optical_frame
- added link support, mass 0.1; collision cylinder length=0.03 radius=0.02; visual cylinder length=0.03 radius=0.02
Joints:
- added joint d435_color_joint: type fixed, parent d435_depth_frame, child d435_color_frame, origin xyz=0 0.015 0 rpy=0 0 0
- added joint d435_color_optical_joint: type fixed, parent d435_color_frame, child d435_color_optical_frame, origin xyz=0 0 0 rpy=-1.5707963267948966 0 -1.5707963267948966
- added joint d435_depth_joint: type fixed, parent d435_link, child d435_depth_frame, origin xyz=0 0 0 rpy=0 0 0
- added joint d435_depth_optical_joint: type fixed, parent d435_depth_frame, child d435_depth_optical_frame, origin xyz=0 0 0 rpy=-1.5707963267948966 0 -1.5707963267948966
- added joint d435_joint: type fixed, parent support, child d435_bottom_screw_frame, origin xyz=0 0 0.01 rpy=0 0 1.57 
- added joint d435_left_ir_joint: type fixed, parent d435_depth_frame, child d435_left_ir_frame, origin xyz=0 0.0 0 rpy=0 0 0
- added joint d435_left_ir_optical_joint: type fixed, parent d435_left_ir_frame, child d435_left_ir_optical_frame, origin xyz=0 0 0 rpy=-1.5707963267948966 0 -1.5707963267948966
- added joint d435_link_joint: type fixed, parent d435_bottom_screw_frame, child d435_link, origin xyz=0 0.0175 0.0125 rpy=0 0 0
- added joint d435_right_ir_joint: type fixed, parent d435_depth_frame, child d435_right_ir_frame, origin xyz=0 -0.05 0 rpy=0 0 0
- added joint d435_right_ir_optical_joint: type fixed, parent d435_right_ir_frame, child d435_right_ir_optical_frame, origin xyz=0 0 0 rpy=-1.5707963267948966 0 -1.5707963267948966
- added joint support2wrist_3_link: type fixed, parent wrist_3_link, child support, origin xyz=0 0.05 0.05
